File: pcb/honda-z50a-regulator.sch (EAGLE design)
At the start: 21 parts, among them CON1 2EDG-2P, CON2 2EDG-2P, Q1 IRF5210, U1 LTC3894

Commit message: Finish PCB Generate gerbers Export PDFs
Parts:
- added C10, C11: 22uF, Capacitor:CAPACITOR-1206
- added C12: 1000uF, Capacitor:ELETROLITIC-CAPACITOR-13MM
- added C13: 1uF, Capacitor:CAPACITOR-1206
- added C8: 1nF, Capacitor:CAPACITOR-0603
- added C9: 10pF, Capacitor:CAPACITOR-0603
- added LOGO1: OSHW-LOGOS, Silkscreen:OSHW-LOGOS
- added LOGO2: JS-5MM, Silkscreen:JS-5MM
- added R7: 0 Ohms, Resistor:RESISTOR-0603
- added R8: 7.15K Ohms, Resistor:RESISTOR-0603
- C1: value 1000uF -> 100uF; device Capacitor:ELETROLITIC-CAPACITOR-13MM -> Capacitor:ELETROLITIC-CAPACITOR-18MM; VOLTAGE 50V -> 400V
- C2: value 100uF -> 220nF; device Capacitor:ELETROLITIC-CAPACITOR-18MM -> Capacitor:CAPACITOR-1206; VOLTAGE 400V -> 200V
- C3: value 100nF -> 1uF; device Capacitor:CAPACITOR-0603 -> Capacitor:CAPACITOR-1206; VOLTAGE (none) -> 100V
- C4: value 3.3nF -> 150pF
- C6: value 1nF -> 1uF; VOLTAGE (none) -> 16V
- C7: VOLTAGE 16V -> (none)
- D1: value MBR5150 -> LED1206; device Generic Diode:MBR5150 -> LED:LED1206
- D2: value LED1206 -> MBR5150; device LED:LED1206 -> Generic Diode:MBR5150
- R1: value 18m Ohms -> 280K Ohms; device Resistor:RESISTOR-2512 -> Resistor:RESISTOR-0603; OCLCSC C270951 -> (none); TOLERANCE 1% -> (none)
- R2: value (none) -> 0 Ohms
- R3: value (none) -> 1.5K Ohms
- R4: value (none) -> 18m Ohms; device Resistor:RESISTOR-0603 -> Resistor:RESISTOR-2512; OCLCSC (none) -> C270951; TOLERANCE (none) -> 1%
- R5: value 5.76K Ohms -> 100K Ohms; device Resistor:RESISTOR-0603 -> Potentiometer:POTENTIOMETER-TH
- R6: value 1.5K Ohms -> 100K Ohms
Connections:
- net N$10 renamed ITH
- net N$11 renamed DRUV
- net N$2 renamed GATE
- removed net N$12: C7.C2, U1.CAP
- removed net N$13: D2.A, R6.1, U1.PGOOD
- removed net N$3: C6.C1, L1.2, R1.2, U1.SENSE+
- removed net N$4: D1.C, L1.1, Q1.D
- removed net N$6: R2.1, R3.2, U1.PGUV, U1.VFB
- removed net N$7: R4.2, U1.FREQ
- removed net N$8: C3.C1, U1.TRACK/SS
- new net CAP: C6.C2, U1.CAP
- new net FREQ: R2.2, U1.FREQ
- new net ISENSE: C8.C1, L1.2, R4.2, U1.SENSE+
- new net N$1: R5.CW, R7.1, R8.2
- new net PGOOD: D1.A, R3.1, U1.PGOOD
- new net SS: C7.C1, U1.TRACK/SS
- new net SW: D2.C, L1.1, Q1.D
- new net VFB: C9.C2, R5.WIPER, R6.1, R7.2, U1.PGUV, U1.VFB
- net 12V0: now also C10.C1, C11.C1, C12.+, C8.C2, C9.C1, R3.2, R4.1; no longer C1.+, C6.C2, R1.1, R2.2
- net GND: now also C10.C2, C11.C2, C12.-, C13.C2, C2.C2, C7.C2, D1.C, D2.A, R1.1, R2.1, R8.1; no longer C2.-, D1.A, D2.C, R3.1, R4.1, R5.1
- net N$9: now also R1.2; no longer R5.2
- net VIN: now also C1.+, C13.C1, C2.C1, C3.C1, C6.C1; no longer C2.+, C7.C1
Other:
- note added: "1 uF = 80 ms"
- moved on the sheet: C1, C2, C3, C4, C5, C6, C7, CON1-1, CON1-2, CON2-1, CON2-2, L1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
