File: pcb/honda-z50a-regulator.brd (EAGLE design)
At the start: 60 x 50 mm, 21 parts, among them CON1 2EDG-2P, CON2 2EDG-2P, Q1 IRF5210, U1 LTC3894

Commit message: Finish PCB Generate gerbers Export PDFs
Parts:
- added C10, C11: 22uF, Capacitor:CAP1206
- added C12: 1000uF, Capacitor:EL-CAP-13MM
- added C13: 1uF, Capacitor:CAP1206
- added C8: 1nF, Capacitor:CAP0603
- added C9: 10pF, Capacitor:CAP0603
- added LOGO1: OSHW-LOGOS, Silkscreen:OSHW-LOGO-S
- added LOGO2: JS-5MM, Silkscreen:JS_5MM
- added R7: 0 Ohms, Resistor:RES0603
- added R8: 7.15K Ohms, Resistor:RES0603
- C1: value 1000uF -> 100uF; device Capacitor:EL-CAP-13MM -> Capacitor:EL-CAP-18MM
- C2: value 100uF -> 220nF; device Capacitor:EL-CAP-18MM -> Capacitor:CAP1206
- C3: value 100nF -> 1uF; device Capacitor:CAP0603 -> Capacitor:CAP1206
- C4: value 3.3nF -> 150pF
- C6: value 1nF -> 1uF
- D1: value MBR5150 -> LED1206; device Generic Diode:DO201AD -> LED:1206
- D2: value LED1206 -> MBR5150; device LED:1206 -> Generic Diode:DO201AD
- R1: value 18m Ohms -> 280K Ohms; device Resistor:RES2512 -> Resistor:RES0603
- R2: value (none) -> 0 Ohms
- R3: value (none) -> 1.5K Ohms
- R4: value (none) -> 18m Ohms; device Resistor:RES0603 -> Resistor:RES2512
- R5: value 5.76K Ohms -> 100K Ohms; device Resistor:RES0603 -> Potentiometer:TRIMMER
- R6: value 1.5K Ohms -> 100K Ohms
- moved D2 77.0 mm to (29.0, 24.0), flipped to the bottom, turned to 180 degrees
- moved C6 76.9 mm to (54.3, 13.4), turned to 270 degrees
- moved SJ1 75.0 mm to (56.2, 9.80)
- moved R6 66.4 mm to (26.5, 7.20), turned to 180 degrees
- moved C7 65.9 mm to (42.9, 3.80), turned to 270 degrees
- moved C3 57.1 mm to (21.9, 36.4), turned to 90 degrees
- moved R2 56.8 mm to (56.2, 7.40), turned to 180 degrees
- moved C5 48.5 mm to (37.5, 3.80), turned to 270 degrees
- moved C4 46.6 mm to (39.3, 3.80), turned to 270 degrees
- moved R3 46.6 mm to (45.8, 3.20), turned to 180 degrees
- moved R5 45.3 mm to (27.8, 3.50), turned to 180 degrees
- moved R4 33.8 mm to (20.0, 15.0), turned to 90 degrees
- moved D1 29.8 mm to (50.3, 3.20), flipped to the top
- moved R1 23.9 mm to (41.1, 3.80), turned to 270 degrees
- moved C1 22.1 mm to (17.0, 36.0)
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Connections:
- net N$10 renamed ITH
- net N$11 renamed DRUV
- net N$2 renamed GATE
- removed net N$12: C7.2, U1.18
- removed net N$13: D2.2, R6.1, U1.12
- removed net N$3: C6.1, L1.2, R1.2, U1.5
- removed net N$4: D1.C, L1.1, Q1.D
- removed net N$6: R2.1, R3.2, U1.8, U1.9
- removed net N$7: R4.2, U1.13
- removed net N$8: C3.1, U1.10
- new net CAP: C6.2, U1.18
- new net FREQ: R2.2, U1.13
- new net ISENSE: C8.1, L1.2, R4.2, U1.5
- new net N$1: R5.E, R7.1, R8.2
- new net PGOOD: D1.2, R3.1, U1.12
- new net SS: C7.1, U1.10
- new net SW: D2.C, L1.1, Q1.D
- new net VFB: C9.2, R5.S, R6.1, R7.2, U1.8, U1.9
- net 12V0: now also C10.1, C11.1, C12.+, C8.2, C9.1, R3.2, R4.1; no longer C1.+, C6.2, R1.1, R2.2
- net GND: now also C10.2, C11.2, C12.-, C13.2, C2.2, C7.2, D1.1, D2.A, R1.1, R2.1, R8.1; no longer C2.-, D1.A, D2.1, R3.1, R4.1, R5.1
- net N$9: now also R1.2; no longer R5.2
- net VIN: now also C1.+, C13.1, C2.1, C3.1, C6.1; no longer C2.+, C7.1
Routing:
- net VIN: track 0.00 -> 63.3 mm, vias 0 -> 2
- net 12V0: track 0.00 -> 59.9 mm, vias 0 -> 4
- net ISENSE: track 0.00 -> 31.2 mm, vias 0 -> 2
- net VFB: track 0.00 -> 30.2 mm, vias 0 -> 2
- net GATE: track 0.00 -> 26.1 mm
- net ITH: track 0.00 -> 9.93 mm
- net PGOOD: track 0.00 -> 9.62 mm, vias 0 -> 2
- net N$1: track 0.00 -> 6.25 mm
- net DRUV: track 0.00 -> 4.51 mm
- net CAP: track 0.00 -> 4.38 mm
- net FREQ: track 0.00 -> 4.02 mm
- net SS: track 0.00 -> 3.33 mm
- net N$9: track 0.00 -> 1.80 mm
- added copper zone on layer 1, net GATE
- added copper zone on layer 1, net ISENSE
- added copper zone on layer 1, net SW
- removed copper zone on layer 1, net N$3
- removed copper zone on layer 1, net N$4
Other:
- outline, holes or cut-outs redrawn
- board text added: "+ -"
- board text added: "Honda Z50A Regulator v1 Dez 2019"
- board text added: "INPUT"
- board text added: "OUTPUT"

Commit message: Sync library updates
Connections:
- net GND: now also D1.C; no longer D1.1
- net PGOOD: now also D1.A; no longer D1.2
